File: bigger_rgb_adapter.sch (KiCad schematic (older format))
At the start: 7 parts, among them J1 Conn_01x10, J2 Conn_01x10

Commit message: Use EAST1616RGBA3 LEDs instead
Parts:
- D1, D2, D3, D4, D5: footprint LED_SMD:LED_Cree-UHD1110-FKA_1x1mm -> LED_SMD:LED_RGB_EAST1616RGBA3
Changed lines of the file:
@@
 EESchema Schematic File Version 4
+LIBS:bigger_rgb_adapter-cache
 EELAYER 29 0
 EELAYER END
@@
 F 0 "D1" V 4546 1220 50  0000 R CNN
 F 1 "LED_BGRA" V 4455 1220 50  0000 R CNN
-F 2 "LED_SMD:LED_Cree-UHD1110-FKA_1x1mm" H 4500 1500 50  0001 C CNN
+F 2 "LED_SMD:LED_RGB_EAST1616RGBA3" H 4500 1500 50  0001 C CNN
 F 3 "~" H 4500 1500 50  0001 C CNN
 	1    4500 1550
@@
 F 0 "D2" V 4546 1770 50  0000 R CNN
 F 1 "LED_BGRA" V 4455 1770 50  0000 R CNN
-F 2 "LED_SMD:LED_Cree-UHD1110-FKA_1x1mm" H 4500 2050 50  0001 C CNN
+F 2 "LED_SMD:LED_RGB_EAST1616RGBA3" H 4500 2050 50  0001 C CNN
 F 3 "~" H 4500 2050 50  0001 C CNN
 	1    4500 2100
@@
 F 0 "D3" V 4546 2370 50  0000 R CNN
 F 1 "LED_BGRA" V 4455 2370 50  0000 R CNN
-F 2 "LED_SMD:LED_Cree-UHD1110-FKA_1x1mm" H 4500 2650 50  0001 C CNN
+F 2 "LED_SMD:LED_RGB_EAST1616RGBA3" H 4500 2650 50  0001 C CNN
 F 3 "~" H 4500 2650 50  0001 C CNN
 	1    4500 2700
@@
 F 0 "D4" V 4546 2920 50  0000 R CNN
 F 1 "LED_BGRA" V 4455 2920 50  0000 R CNN
-F 2 "LED_SMD:LED_Cree-UHD1110-FKA_1x1mm" H 4500 3200 50  0001 C CNN
+F 2 "LED_SMD:LED_RGB_EAST1616RGBA3" H 4500 3200 50  0001 C CNN
 F 3 "~" H 4500 3200 50  0001 C CNN
 	1    4500 3250
@@
 F 0 "D5" V 4546 3570 50  0000 R CNN
 F 1 "LED_BGRA" V 4455 3570 50  0000 R CNN
-F 2 "LED_SMD:LED_Cree-UHD1110-FKA_1x1mm" H 4500 3850 50  0001 C CNN
+F 2 "LED_SMD:LED_RGB_EAST1616RGBA3" H 4500 3850 50  0001 C CNN
 F 3 "~" H 4500 3850 50  0001 C CNN
 	1    4500 3900
@@
 	2900 2350 2500 2350
 Wire Wire Line
-	4500 1350 2850 1350
-Wire Wire Line
 	2850 1350 2850 2250
 Wire Wire Line
@@
 	3000 2550 2500 2550
 Wire Wire Line
-	4500 1900 2950 1900
-Wire Wire Line
 	2950 1900 2950 2450
 Wire Wire Line
 	2950 2450 2500 2450
 Wire Wire Line
-	4500 2500 3050 2500
-Wire Wire Line
 	3050 2500 3050 2650
 Wire Wire Line
@@
 	4000 3050 4000 2850
 Wire Wire Line
-	4000 2850 2500 2850
-Wire Wire Line
 	4300 3450 3950 3450
 Wire Wire Line
@@
 	3900 3700 3900 3050
 Wire Wire Line
-	3900 3050 2500 3050
-Wire Wire Line
 	4300 4100 3850 4100
 Wire Wire Line
@@
 Wire Wire Line
 	5450 3150 6450 3150
+Wire Wire Line
+	2850 1350 4500 1350
+Wire Wire Line
+	2950 1900 4500 1900
+Wire Wire Line
+	3050 2500 4500 2500
+Wire Wire Line
+	2500 3050 3900 3050
+Wire Wire Line
+	2500 2850 4000 2850
 $EndSCHEMATC
